File: Sofle_Extended.kicad_pcb (KiCad board)
At the start: 2 copper layers, 166.7 x 142.9 mm, 108 parts, among them J1 LED-Lily58-cache, J2 OLED-Lily58-cache, J3 SofleKeyboard-rescue_MJ-4PP-9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, SW1 SW_PUSH, SW10 SW_PUSH, SW11 SW_PUSH, SW12 SW_PUSH, SW13 SW_PUSH, SW14 SW_PUSH, SW15 SW_PUSH, SW16 SW_PUSH, SW17 SW_PUSH, SW18 SW_PUSH, SW19 SW_PUSH, SW2 SW_PUSH, SW20 SW_PUSH, SW21 SW_PUSH, SW22 SW_PUSH, SW23 SW_PUSH, SW24 SW_PUSH, SW25 SW_PUSH, SW26 SW_PUSH, SW27 SW_PUSH, SW28 SW_PUSH, SW29 SW_PUSH, SW3 SW_PUSH, SW30 SW_PUSH, SW31 SW_PUSH, SW32 SW_PUSH, SW33 SW_PUSH, SW34 SW_PUSH, SW35 SW_PUSH, SW36 SW_PUSH, SW37 SW_PUSH, SW38 SW_PUSH, SW39 SW_PUSH, SW4 SW_PUSH, SW40 SW_PUSH, SW41 SW_PUSH, SW42 Device_Rotary_Encoder_Switch, SW5 SW_PUSH, SW6 SW_PUSH, SW7 SW_PUSH, SW8 SW_PUSH, SW9 SW_PUSH, U1 Elite-C

Commit message: Add V1.1 design files
Parts:
- added TH8: HOLE, SofleKeyboard-footprint:HOLE_M2_TH, F.Cu at (78.0, 97.5)
- moved J3 64.8 mm to (66.9, 36.8), turned to 0 degrees
- moved TH1 27.3 mm to (76.0, 83.8)
- moved TH2 27.3 mm to (86.4, 83.8)
- moved RSW1 22.7 mm to (66.0, 71.8), turned to 90 degrees
- moved J2 4.13 mm to (77.2, 73.7)
- moved JP1 4.13 mm to (84.9, 69.7)
- moved JP2 4.13 mm to (82.5, 69.7)
- moved JP3 4.13 mm to (79.4, 69.7)
- moved JP4 4.13 mm to (77.0, 69.7)
- moved JP5 4.13 mm to (84.9, 69.7)
- moved JP6 4.13 mm to (82.5, 69.7)
- moved JP7 4.13 mm to (79.4, 69.7)
- moved JP8 4.13 mm to (77.0, 69.7)
Routing:
- net col0: track 277.4 -> 345.7 mm, vias 7 -> 10
- net col1: track 265.6 -> 328.6 mm, vias 6 -> 9
- net /i2c_c: track 66.0 -> 24.0 mm, vias 1 -> 0
- net RESET: track 80.1 -> 45.3 mm
- net /i2c_d: track 63.7 -> 32.7 mm, vias 3 -> 1
- net VCC: track 106.2 -> 87.9 mm, vias 4 -> 2
- net ENCB: track 112.3 -> 94.5 mm, vias 1 -> 4
- net GND: track 181.3 -> 166.4 mm, vias 3 -> 2
- net col4: track 199.0 -> 211.7 mm, vias 8 -> 12
- net LED: track 83.0 -> 92.6 mm
- net col3: track 211.2 -> 219.3 mm, vias 9 -> 10
- net SW25A: track 114.9 -> 107.6 mm
- net col2: track 226.8 -> 232.5 mm, vias 9 -> 8
- net Net-(D24-Pad2): track 21.4 -> 26.4 mm
- net Net-(D17-Pad2): track 21.3 -> 26.3 mm
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