File: Sofle_Extended.kicad_sch (KiCad schematic)
At the start: 108 parts, among them J1 LED-Lily58-cache, J2 OLED-Lily58-cache, J3 SofleKeyboard-rescue_MJ-4PP-9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, SW1 SW_PUSH, SW10 SW_PUSH, SW11 SW_PUSH, SW12 SW_PUSH, SW13 SW_PUSH, SW14 SW_PUSH, SW15 SW_PUSH, SW16 SW_PUSH, SW17 SW_PUSH, SW18 SW_PUSH, SW19 SW_PUSH, SW2 SW_PUSH, SW20 SW_PUSH, SW21 SW_PUSH, SW22 SW_PUSH, SW23 SW_PUSH, SW24 SW_PUSH, SW25 SW_PUSH, SW26 SW_PUSH, SW27 SW_PUSH, SW28 SW_PUSH, SW29 SW_PUSH, SW3 SW_PUSH, SW30 SW_PUSH, SW31 SW_PUSH, SW32 SW_PUSH, SW33 SW_PUSH, SW34 SW_PUSH, SW35 SW_PUSH, SW36 SW_PUSH, SW37 SW_PUSH, SW38 SW_PUSH, SW39 SW_PUSH, SW4 SW_PUSH, SW40 SW_PUSH, SW41 SW_PUSH, SW42 Device_Rotary_Encoder_Switch, SW5 SW_PUSH, SW6 SW_PUSH, SW7 SW_PUSH, SW8 SW_PUSH, SW9 SW_PUSH, U1 Elite-C

Commit message: Add V1.1 design files
Parts:
- added TH8: HOLE, SofleKeyboard-footprint:HOLE_M2_TH, symbol SofleKeyboard-rescue:HOLE-Lily58-cache-Lily58_Pro-rescue
Other:
- moved on the sheet: TH1, TH2, TH3, TH4, TH5, TH6, TH7
Changed lines of the file:
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@@
     (pin "2")
   )
-  (symbol (lib_id "SofleKeyboard-rescue:HOLE-Lily58-cache-Lily58_Pro-rescue") (at 252.73 160.02 0) (unit 1)
-    (in_bom yes) (on_board yes)
-    (property "Reference" "TH7" (id 0) (at 252.73 160.02 0)
-      (effects (font (size 1.524 1.524)))
-    )
-    (property "Value" "HOLE" (id 1) (at 252.73 162.56 0)
-      (effects (font (size 1.524 1.524)))
-    )
-    (property "Footprint" "SofleKeyboard-footprint:HOLE_M2_TH" (id 2) (at 252.73 160.02 0)
+  (symbol (lib_id "SofleKeyboard-rescue:HOLE-Lily58-cache-Lily58_Pro-rescue") (at 234.95 160.02 0) (unit 1)
+    (in_bom yes) (on_board yes)
+    (property "Reference" "TH7" (id 0) (at 234.95 160.02 0)
+      (effects (font (size 1.524 1.524)))
+    )
+    (property "Value" "HOLE" (id 1) (at 234.95 162.56 0)
+      (effects (font (size 1.524 1.524)))
+    )
+    (property "Footprint" "SofleKeyboard-footprint:HOLE_M2_TH" (id 2) (at 234.95 160.02 0)
       (effects (font (size 1.524 1.524)) hide)
     )
-    (property "Datasheet" "" (id 3) (at 252.73 160.02 0)
+    (property "Datasheet" "" (id 3) (at 234.95 160.02 0)
       (effects (font (size 1.524 1.524)))
     )
@@
     (pin "2")
   )
+  (symbol (lib_id "SofleKeyboard-rescue:HOLE-Lily58-cache-Lily58_Pro-rescue") (at 243.84 160.02 0) (unit 1)
+    (in_bom yes) (on_board yes)
+    (property "Reference" "TH8" (id 0) (at 243.84 160.02 0)
+      (effects (font (size 1.524 1.524)))
+    )
+    (property "Value" "HOLE" (id 1) (at 243.84 162.56 0)
+      (effects (font (size 1.524 1.524)))
+    )
+    (property "Footprint" "SofleKeyboard-footprint:HOLE_M2_TH" (id 2) (at 243.84 160.02 0)
+      (effects (font (size 1.524 1.524)) hide)
+    )
+    (property "Datasheet" "" (id 3) (at 243.84 160.02 0)
+      (effects (font (size 1.524 1.524)))
+    )
+  )
   (symbol (lib_id "SofleKeyboard-rescue:D-Lily58-cache-Lily58_Pro-rescue") (at 152.4 78.74 90) (unit 1)
     (in_bom yes) (on_board yes)
@@
     (pin "2")
   )
-  (symbol (lib_id "SofleKeyboard-rescue:HOLE-Lily58-cache-Lily58_Pro-rescue") (at 243.84 160.02 0) (unit 1)
-    (in_bom yes) (on_board yes)
-    (property "Reference" "TH6" (id 0) (at 243.84 160.02 0)
-      (effects (font (size 1.524 1.524)))
-    )
-    (property "Value" "HOLE" (id 1) (at 243.84 162.56 0)
-      (effects (font (size 1.524 1.524)))
-    )
-    (property "Footprint" "SofleKeyboard-footprint:HOLE_M2_TH" (id 2) (at 243.84 160.02 0)
+  (symbol (lib_id "SofleKeyboard-rescue:HOLE-Lily58-cache-Lily58_Pro-rescue") (at 226.06 160.02 0) (unit 1)
+    (in_bom yes) (on_board yes)
+    (property "Reference" "TH6" (id 0) (at 226.06 160.02 0)
+      (effects (font (size 1.524 1.524)))
+    )
+    (property "Value" "HOLE" (id 1) (at 226.06 162.56 0)
+      (effects (font (size 1.524 1.524)))
+    )
+    (property "Footprint" "SofleKeyboard-footprint:HOLE_M2_TH" (id 2) (at 226.06 160.02 0)
       (effects (font (size 1.524 1.524)) hide)
     )
-    (property "Datasheet" "" (id 3) (at 243.84 160.02 0)
-      (effects (font (size 1.524 1.524)))
-    )
-  )
-  (symbol (lib_id "SofleKeyboard-rescue:HOLE-Lily58-cache-Lily58_Pro-rescue") (at 191.77 160.02 0) (unit 1)
-    (in_bom yes) (on_board yes)
-    (property "Reference" "TH1" (id 0) (at 191.77 160.02 0)
-      (effects (font (size 1.524 1.524)))
-    )
-    (property "Value" "HOLE" (id 1) (at 191.77 162.56 0)
-      (effects (font (size 1.524 1.524)))
-    )
-    (property "Footprint" "SofleKeyboard-footprint:M2_HOLE_PCB" (id 2) (at 191.77 160.02 0)
+    (property "Datasheet" "" (id 3) (at 226.06 160.02 0)
+      (effects (font (size 1.524 1.524)))
+    )
+  )
+  (symbol (lib_id "SofleKeyboard-rescue:HOLE-Lily58-cache-Lily58_Pro-rescue") (at 181.61 160.02 0) (unit 1)
+    (in_bom yes) (on_board yes)
+    (property "Reference" "TH1" (id 0) (at 181.61 160.02 0)
+      (effects (font (size 1.524 1.524)))
+    )
+    (property "Value" "HOLE" (id 1) (at 181.61 162.56 0)
+      (effects (font (size 1.524 1.524)))
+    )
+    (property "Footprint" "SofleKeyboard-footprint:M2_HOLE_PCB" (id 2) (at 181.61 160.02 0)
       (effects (font (size 1.524 1.524)) hide)
     )
-    (property "Datasheet" "" (id 3) (at 191.77 160.02 0)
+    (property "Datasheet" "" (id 3) (at 181.61 160.02 0)
       (effects (font (size 1.524 1.524)))
     )
@@
     (pin "2")
   )
-  (symbol (lib_id "SofleKeyboard-rescue:HOLE-Lily58-cache-Lily58_Pro-rescue") (at 217.17 160.02 0) (unit 1)
-    (in_bom yes) (on_board yes)
-    (property "Reference" "TH3" (id 0) (at 217.17 160.02 0)
-      (effects (font (size 1.524 1.524)))
-    )
-    (property "Value" "HOLE" (id 1) (at 217.17 162.56 0)
-      (effects (font (size 1.524 1.524)))
-    )
-    (property "Footprint" "SofleKeyboard-footprint:HOLE_M2_TH" (id 2) (at 217.17 160.02 0)
+  (symbol (lib_id "SofleKeyboard-rescue:HOLE-Lily58-cache-Lily58_Pro-rescue") (at 199.39 160.02 0) (unit 1)
+    (in_bom yes) (on_board yes)
+    (property "Reference" "TH3" (id 0) (at 199.39 160.02 0)
+      (effects (font (size 1.524 1.524)))
+    )
+    (property "Value" "HOLE" (id 1) (at 199.39 162.56 0)
+      (effects (font (size 1.524 1.524)))
+    )
+    (property "Footprint" "SofleKeyboard-footprint:HOLE_M2_TH" (id 2) (at 199.39 160.02 0)
       (effects (font (size 1.524 1.524)) hide)
     )
-    (property "Datasheet" "" (id 3) (at 217.17 160.02 0)
+    (property "Datasheet" "" (id 3) (at 199.39 160.02 0)
       (effects (font (size 1.524 1.524)))
     )
@@
     (pin "1")
   )
-  (symbol (lib_id "SofleKeyboard-rescue:HOLE-Lily58-cache-Lily58_Pro-rescue") (at 234.95 160.02 0) (unit 1)
-    (in_bom yes) (on_board yes)
-    (property "Reference" "TH5" (id 0) (at 234.95 160.02 0)
-      (effects (font (size 1.524 1.524)))
-    )
-    (property "Value" "HOLE" (id 1) (at 234.95 162.56 0)
-      (effects (font (size 1.524 1.524)))
-    )
-    (property "Footprint" "SofleKeyboard-footprint:HOLE_M2_TH" (id 2) (at 234.95 160.02 0)
+  (symbol (lib_id "SofleKeyboard-rescue:HOLE-Lily58-cache-Lily58_Pro-rescue") (at 217.17 160.02 0) (unit 1)
+    (in_bom yes) (on_board yes)
+    (property "Reference" "TH5" (id 0) (at 217.17 160.02 0)
+      (effects (font (size 1.524 1.524)))
+    )
+    (property "Value" "HOLE" (id 1) (at 217.17 162.56 0)
+      (effects (font (size 1.524 1.524)))
+    )
+    (property "Footprint" "SofleKeyboard-footprint:HOLE_M2_TH" (id 2) (at 217.17 160.02 0)
       (effects (font (size 1.524 1.524)) hide)
     )
-    (property "Datasheet" "" (id 3) (at 234.95 160.02 0)
+    (property "Datasheet" "" (id 3) (at 217.17 160.02 0)
       (effects (font (size 1.524 1.524)))
     )
@@
     (pin "1")
   )
-  (symbol (lib_id "SofleKeyboard-rescue:HOLE-Lily58-cache-Lily58_Pro-rescue") (at 226.06 160.02 0) (unit 1)
-    (in_bom yes) (on_board yes)
-    (property "Reference" "TH4" (id 0) (at 226.06 160.02 0)
-      (effects (font (size 1.524 1.524)))
-    )
-    (property "Value" "HOLE" (id 1) (at 226.06 162.56 0)
-      (effects (font (size 1.524 1.524)))
-    )
-    (property "Footprint" "SofleKeyboard-footprint:HOLE_M2_TH" (id 2) (at 226.06 160.02 0)
+  (symbol (lib_id "SofleKeyboard-rescue:HOLE-Lily58-cache-Lily58_Pro-rescue") (at 208.28 160.02 0) (unit 1)
+    (in_bom yes) (on_board yes)
+    (property "Reference" "TH4" (id 0) (at 208.28 160.02 0)
+      (effects (font (size 1.524 1.524)))
+    )
+    (property "Value" "HOLE" (id 1) (at 208.28 162.56 0)
+      (effects (font (size 1.524 1.524)))
+    )
+    (property "Footprint" "SofleKeyboard-footprint:HOLE_M2_TH" (id 2) (at 208.28 160.02 0)
       (effects (font (size 1.524 1.524)) hide)
     )
-    (property "Datasheet" "" (id 3) (at 226.06 160.02 0)
+    (property "Datasheet" "" (id 3) (at 208.28 160.02 0)
       (effects (font (size 1.524 1.524)))
     )
@@
     (pin "2")
   )
-  (symbol (lib_id "SofleKeyboard-rescue:HOLE-Lily58-cache-Lily58_Pro-rescue") (at 200.66 160.02 0) (unit 1)
-    (in_bom yes) (on_board yes)
-    (property "Reference" "TH2" (id 0) (at 200.66 160.02 0)
-      (effects (font (size 1.524 1.524)))
-    )
-    (property "Value" "HOLE" (id 1) (at 200.66 162.56 0)
-      (effects (font (size 1.524 1.524)))
-    )
-    (property "Footprint" "SofleKeyboard-footprint:M2_HOLE_PCB" (id 2) (at 200.66 160.02 0)
+  (symbol (lib_id "SofleKeyboard-rescue:HOLE-Lily58-cache-Lily58_Pro-rescue") (at 190.5 160.02 0) (unit 1)
+    (in_bom yes) (on_board yes)
+    (property "Reference" "TH2" (id 0) (at 190.5 160.02 0)
+      (effects (font (size 1.524 1.524)))
+    )
+    (property "Value" "HOLE" (id 1) (at 190.5 162.56 0)
+      (effects (font (size 1.524 1.524)))
+    )
+    (property "Footprint" "SofleKeyboard-footprint:M2_HOLE_PCB" (id 2) (at 190.5 160.02 0)
       (effects (font (size 1.524 1.524)) hide)
     )
-    (property "Datasheet" "" (id 3) (at 200.66 160.02 0)
+    (property "Datasheet" "" (id 3) (at 190.5 160.02 0)
       (effects (font (size 1.524 1.524)))
     )
@@
       (reference "TH7") (unit 1) (value "HOLE") (footprint "SofleKeyboard-footprint:HOLE_M2_TH")
     )
+    (path "/5d298953-216c-4fc2-a9ee-ca3fc245ca6e"
+      (reference "TH8") (unit 1) (value "HOLE") (footprint "SofleKeyboard-footprint:HOLE_M2_TH")
+    )
     (path "/4cafb73d-1ad8-4d24-acf7-63d78095ae46"
